Commit message: add 3 cameras

File: turtlebot3_description/urdf/turtlebot3_waffle_pi.gazebo.xacro (robot description, xacro)
@@ -135,10 +135,44 @@
   </gazebo>
 <!--link : https://www.raspberrypi.org/documentation/hardware/camera/-->
-  <gazebo reference="camera_rgb_frame">
-    <sensor type="camera" name="Pi Camera">
+  <gazebo reference="camera_rgb_left_frame">
+    <sensor type="camera" name="camera_left">
       <always_on>true</always_on>
       <visualize>$(arg camera_visual)</visualize>
       <camera>
-          <horizontal_fov>1.085595</horizontal_fov>
+          <horizontal_fov>2.09</horizontal_fov>
+          <image>
+              <width>640</width>
+              <height>480</height>
+              <format>R8G8B8</format>
+          </image>
+          <clip>
+              <near>0.03</near>
+              <far>100</far>
+          </clip>
+      </camera>
+      <plugin name="camera_controller" filename="libgazebo_ros_camera.so">
+		<topicName>camera_left</topicName>
+		<alwaysOn>true</alwaysOn>
+        <updateRate>30.0</updateRate>
+        <cameraName>camera_left</cameraName>
+        <frameName>camera_rgb_optical_left_frame</frameName>
+        <imageTopicName>rgb/image_raw</imageTopicName>
+        <cameraInfoTopicName>rgb/camera_info</cameraInfoTopicName>
+        <hackBaseline>0.07</hackBaseline>
+        <distortionK1>0.0</distortionK1>
+        <distortionK2>0.0</distortionK2>
+        <distortionK3>0.0</distortionK3>
+        <distortionT1>0.0</distortionT1>
+        <distortionT2>0.0</distortionT2>
+      </plugin>
+    </sensor>
+  </gazebo>
+<!--link : https://www.raspberrypi.org/documentation/hardware/camera/-->
+  <gazebo reference="camera_rgb_frame">
+    <sensor type="camera" name="camera">
+      <always_on>true</always_on>
+      <visualize>$(arg camera_visual)</visualize>
+      <camera>
+          <horizontal_fov>2.09</horizontal_fov>
           <image>
               <width>640</width>
@@ -167,3 +201,37 @@
     </sensor>
   </gazebo>
+<!--link : https://www.raspberrypi.org/documentation/hardware/camera/-->
+  <gazebo reference="camera_rgb_right_frame">
+    <sensor type="camera" name="camera_right">
+      <always_on>true</always_on>
+      <visualize>$(arg camera_visual)</visualize>
+      <camera>
+          <horizontal_fov>2.09</horizontal_fov>
+          <image>
+              <width>640</width>
+              <height>480</height>
+              <format>R8G8B8</format>
+          </image>
+          <clip>
+              <near>0.03</near>
+              <far>100</far>
+          </clip>
+      </camera>
+      <plugin name="camera_controller" filename="libgazebo_ros_camera.so">
+        <topicName>camera_right</topicName>
+        <alwaysOn>true</alwaysOn>
+        <updateRate>30.0</updateRate>
+        <cameraName>camera_right</cameraName>
+        <frameName>camera_rgb_optical_right_frame</frameName>
+        <imageTopicName>rgb/image_raw</imageTopicName>
+        <cameraInfoTopicName>rgb/camera_info</cameraInfoTopicName>
+        <hackBaseline>0.07</hackBaseline>
+        <distortionK1>0.0</distortionK1>
+        <distortionK2>0.0</distortionK2>
+        <distortionK3>0.0</distortionK3>
+        <distortionT1>0.0</distortionT1>
+        <distortionT2>0.0</distortionT2>
+      </plugin>
+    </sensor>
+  </gazebo>
 </robot>

File: turtlebot3_description/urdf/turtlebot3_waffle_pi.urdf.xacro (robot description, xacro)
@@ -161,5 +161,5 @@
   </link>
   <joint name="camera_joint" type="fixed">
-    <origin xyz="0.073 -0.011 0.084" rpy="0 0 0"/>
+    <origin xyz="0.073 -0.011 0.384" rpy="0 0.524 0"/>
     <parent link="base_link"/>
     <child link="camera_link"/>
@@ -185,3 +185,27 @@
   </joint>
   <link name="camera_rgb_optical_frame"/>
+  <joint name="camera_rgb_left_joint" type="fixed">
+    <origin xyz="0.003 0.111 0.009" rpy="0 0 0.175"/>
+    <parent link="camera_link"/>
+    <child link="camera_rgb_left_frame"/>
+  </joint>
+  <link name="camera_rgb_left_frame"/>
+  <joint name="camera_rgb_optical_left_joint" type="fixed">
+    <origin xyz="0 0 0" rpy="-1.57 0 -1.57"/>
+    <parent link="camera_rgb_left_frame"/>
+    <child link="camera_rgb_optical_left_frame"/>
+  </joint>
+  <link name="camera_rgb_optical_left_frame"/>
+  <joint name="camera_rgb_right_joint" type="fixed">
+    <origin xyz="0.003 -0.089 0.009" rpy="0 0 -0.175"/>
+    <parent link="camera_link"/>
+    <child link="camera_rgb_right_frame"/>
+  </joint>
+  <link name="camera_rgb_right_frame"/>
+  <joint name="camera_rgb_optical_right_joint" type="fixed">
+    <origin xyz="0 0 0" rpy="-1.57 0 -1.57"/>
+    <parent link="camera_rgb_right_frame"/>
+    <child link="camera_rgb_optical_right_frame"/>
+  </joint>
+  <link name="camera_rgb_optical_right_frame"/>
 </robot>

Commit message: update for stereo camera

File: turtlebot3_description/urdf/turtlebot3_waffle_pi.gazebo.xacro (robot description, xacro)
@@ -152,11 +152,11 @@
       </camera>
       <plugin name="camera_controller" filename="libgazebo_ros_camera.so">
-		<topicName>camera_left</topicName>
+		<topicName>stereo/left</topicName>
 		<alwaysOn>true</alwaysOn>
         <updateRate>30.0</updateRate>
-        <cameraName>camera_left</cameraName>
+        <cameraName>stereo/left</cameraName>
         <frameName>camera_rgb_optical_left_frame</frameName>
-        <imageTopicName>rgb/image_raw</imageTopicName>
-        <cameraInfoTopicName>rgb/camera_info</cameraInfoTopicName>
+        <imageTopicName>image_raw</imageTopicName>
+        <cameraInfoTopicName>camera_info</cameraInfoTopicName>
         <hackBaseline>0.07</hackBaseline>
         <distortionK1>0.0</distortionK1>
@@ -219,11 +219,11 @@
       </camera>
       <plugin name="camera_controller" filename="libgazebo_ros_camera.so">
-        <topicName>camera_right</topicName>
+        <topicName>stereo/right</topicName>
         <alwaysOn>true</alwaysOn>
         <updateRate>30.0</updateRate>
-        <cameraName>camera_right</cameraName>
+        <cameraName>stereo/right</cameraName>
         <frameName>camera_rgb_optical_right_frame</frameName>
-        <imageTopicName>rgb/image_raw</imageTopicName>
-        <cameraInfoTopicName>rgb/camera_info</cameraInfoTopicName>
+        <imageTopicName>image_raw</imageTopicName>
+        <cameraInfoTopicName>camera_info</cameraInfoTopicName>
         <hackBaseline>0.07</hackBaseline>
         <distortionK1>0.0</distortionK1>

File: turtlebot3_description/urdf/turtlebot3_waffle_pi.urdf.xacro (robot description, xacro)
@@ -173,4 +173,16 @@
     </collision>
   </link>
+  <joint name="camera_rgb_left_joint" type="fixed">
+    <origin xyz="0.003 0.111 0.009" rpy="0 0 0"/>
+    <parent link="camera_link"/>
+    <child link="camera_rgb_left_frame"/>
+  </joint>
+  <link name="camera_rgb_left_frame"/>
+  <joint name="camera_rgb_optical_left_joint" type="fixed">
+    <origin xyz="0 0 0" rpy="-1.57 0 -1.57"/>
+    <parent link="camera_rgb_left_frame"/>
+    <child link="camera_rgb_optical_left_frame"/>
+  </joint>
+  <link name="camera_rgb_optical_left_frame"/>
   <joint name="camera_rgb_joint" type="fixed">
     <origin xyz="0.003 0.011 0.009" rpy="0 0 0"/>
@@ -185,18 +197,6 @@
   </joint>
   <link name="camera_rgb_optical_frame"/>
-  <joint name="camera_rgb_left_joint" type="fixed">
-    <origin xyz="0.003 0.111 0.009" rpy="0 0 0.175"/>
-    <parent link="camera_link"/>
-    <child link="camera_rgb_left_frame"/>
-  </joint>
-  <link name="camera_rgb_left_frame"/>
-  <joint name="camera_rgb_optical_left_joint" type="fixed">
-    <origin xyz="0 0 0" rpy="-1.57 0 -1.57"/>
-    <parent link="camera_rgb_left_frame"/>
-    <child link="camera_rgb_optical_left_frame"/>
-  </joint>
-  <link name="camera_rgb_optical_left_frame"/>
   <joint name="camera_rgb_right_joint" type="fixed">
-    <origin xyz="0.003 -0.089 0.009" rpy="0 0 -0.175"/>
+    <origin xyz="0.003 -0.089 0.009" rpy="0 0 0"/>
     <parent link="camera_link"/>
     <child link="camera_rgb_right_frame"/>
